Commit message: added movement of second joint

File: robotiq/robotiq_s_model_visualization/cfg/robotiq_hand_macro.urdf.xacro (robot description, xacro)
@@ -20,13 +20,4 @@
         </material>
       </visual>
-      <collision>
-        <origin rpy="0 0 0" xyz="0 0 0"/>
-        <geometry>
-          <mesh filename="package://robotiq_s_model_visualization/meshes/s-model_articulated/collision/link_0.STL" />
-        </geometry>
-        <material name="yellow">
-          <color rgba="0 1 1 1"/>
-        </material>
-      </collision>
       <inertial>
         <mass value="0.1"/>
@@ -48,13 +39,4 @@
         <material name="green"/>
       </visual>
-      <collision>
-        <origin rpy="0 0 ${3.1416/2}" xyz="0 0.05717 0"/>
-        <geometry>
-          <mesh filename="package://robotiq_s_model_visualization/meshes/s-model_articulated/collision/link_1.STL"/>
-        </geometry>
-        <material name="yellow">
-          <color rgba="0 1 1 1"/>
-        </material>
-      </collision>
       <inertial>
         <origin rpy="0 0 ${3.1416/2}" xyz="0.00053 0.03218 0"/>
@@ -81,11 +63,4 @@
         <material name="green"/>
       </visual>
-      <collision>
-        <origin rpy="0 0 ${3.1416/2}" xyz="0 0.03810 0.0075"/>
-          <geometry>
-            <mesh filename="package://robotiq_s_model_visualization/meshes/s-model_articulated/collision/link_2.STL"/>
-          </geometry>
-        <material name="yellow"/>
-      </collision>
       <inertial>
         <origin rpy="0 0 ${3.1416/2}" xyz="0.00048 0.02167 0.00018"/>
@@ -112,11 +87,4 @@
         <material name="green"/>
       </visual>
-      <collision>
-        <origin xyz="0 0 0" rpy="0 0 0"/>
-        <geometry>
-          <mesh filename="package://robotiq_s_model_visualization/meshes/s-model_articulated/collision/link_3.STL"/>
-        </geometry>
-        <material name="yellow"/>
-      </collision>
       <inertial>
         <origin rpy="0 0 0" xyz="0.01626 0.00049 0.0002"/>
@@ -135,372 +103,26 @@
     </gazebo>
     <!-- Link proximal actuating hinge -->
-    <link name="${prefix}link_proximal_actuating_hinge">
-      <visual>
-        <origin rpy="0 0 0" xyz="0.01429 0 0"/>
-        <geometry>
-          <box size="0.02858 .0075 .002"/>
-        </geometry>
-      </visual>
-      <collision>
-        <origin rpy="0 0 0" xyz="0.01429 0 0"/>
-         <geometry>
-          <box size="0.02858 .0075 .002"/>
-        </geometry>
-      </collision>
-      <inertial>
-        <origin rpy="0 0 0" xyz="0.0012 -0.00162 -0.00161"/>
-        <mass value="0.02647"/>
-        <inertia ixx= "0.00000156447"
-                 ixy= "0.000000236226"
-                 ixz="-0.00000014862"
-                 iyy= "0.00000221068"
-                 iyz="-0.00000014369"
-                 izz= "0.00000323175"/>
-      </inertial>
-    </link>
-    <gazebo reference="${prefix}link_proximal_actuating_hinge">
-      <mu1>1.1</mu1>
-      <mu2>1.1</mu2>
-    </gazebo>
     <!-- Link paraproximal actuating hinge -->
-    <link name="${prefix}link_paraproximal_actuating_hinge">
-      <visual>
-        <origin rpy="0 0 0" xyz="0.01143 0 0"/>
-        <geometry>
-          <box size="0.02286 .0075 .002"/>
-        </geometry>
-      </visual>
-      <collision>
-        <origin rpy="0 0 0" xyz="0.01143 0 0"/>
-         <geometry>
-          <box size="0.02286 .0075 .002"/>
-        </geometry>
-      </collision>
-      <inertial>
-        <origin rpy="0 0 0" xyz="0.0064 0 0"/>
-        <!-- copied from proximal_actuating_hinge -->
-        <mass value="0.00362"/>
-        <inertia ixx= "0.00000012043"
-                 ixy= "0"
-                 ixz= "0"
-                 iyy= "0.00000053588"
-                 iyz= "0"
-                 izz= "0.00000065322"/>
-      </inertial>
-    </link>
-    <gazebo reference="${prefix}link_paraproximal_actuating_hinge">
-      <mu1>1.1</mu1>
-      <mu2>1.1</mu2>
-    </gazebo>
     <!-- Link proximal actuating bar -->
-    <link name="${prefix}link_proximal_actuating_bar">
-      <visual>
-        <origin rpy="0 0 0" xyz="0.026789 0 0"/>
-        <geometry>
-          <box size="0.05398 .0075 .002"/>
-        </geometry>
-      </visual>
-      <collision>
-        <origin rpy="0 0 0" xyz="0.026789 0 0"/>
-         <geometry>
-          <box size="0.05398 .0075 .002"/>
-        </geometry>
-      </collision>
-      <inertial>
-        <origin rpy="0 0 0" xyz="0.02699 -0.00122 0"/>
-        <mass value="0.00659"/>
-        <inertia ixx= "0.00000008348"
-                 ixy="-0.0000002179"
-                 ixz= "0.00000000134"
-                 iyy= "0.00000719076"
-                 iyz= "0"
-                 izz= "0.00000718272"/>
-      </inertial>
-    </link>
-    <gazebo reference="${prefix}link_proximal_actuating_bar">
-      <mu1>1.1</mu1>
-      <mu2>1.1</mu2>
-    </gazebo>
     <!-- Link paraproximal bar -->
-    <link name="${prefix}link_paraproximal_bar">
-      <visual>
-        <origin rpy="0 0 0" xyz="0.02885 0 0"/>
-        <geometry>
-          <box size="0.05770 .0075 .002"/>
-        </geometry>
-      </visual>
-      <collision>
-        <origin rpy="0 0 0" xyz="0.02885 0 0"/>
-         <geometry>
-          <box size="0.05770 .0075 .002"/>
-        </geometry>
-      </collision>
-      <inertial>
-        <origin rpy="0 0 0" xyz="0.02858 -0.00129 0"/>
-        <mass value="0.00732"/>
-        <inertia ixx= "0.00000009065"
-                 ixy="-0.00000027047"
-                 ixz= "0.00000000142"
-                 iyy= "0.00000878034"
-                 iyz= "0"
-                 izz= "0.00000877558"/>
-      </inertial>
-    </link>
-    <gazebo reference="${prefix}link_paraproximal_bar">
-      <mu1>1.1</mu1>
-      <mu2>1.1</mu2>
-    </gazebo>
     <!-- Link median actuating hinge -->
-    <link name="${prefix}link_median_actuating_hinge">
-      <visual>
-        <origin rpy="0 0 0" xyz="0 0 0"/>
-        <geometry>
-          <box size=".02 .02 .002"/>
-        </geometry>
-      </visual>
-      <collision>
-        <origin rpy="0 0 0" xyz="0 0 0"/>
-         <geometry>
-          <box size=".02 .02 .002"/>
-        </geometry>
-      </collision>
-      <inertial>
-        <origin rpy="0 0 0" xyz="0.0092 0.00514 0"/>
-        <mass value="0.00359"/>
-        <inertia ixx= "0.00000024735"
-                 ixy= "0.00000023619"
-                 ixz= "0"
-                 iyy= "0.00000047681"
-                 iyz= "0"
-                 izz= "0.00000071813"/>
-      </inertial>
-    </link>
-    <gazebo reference="${prefix}link_median_actuating_hinge">
-      <mu1>1.1</mu1>
-      <mu2>1.1</mu2>
-    </gazebo>
     <!-- Link median bar -->
-    <link name="${prefix}link_median_bar">
-      <visual>
-        <origin rpy="0 0 0" xyz="0.01905 0 0"/>
-        <geometry>
-          <box size="0.0381 .0075 .002"/>
-        </geometry>
-      </visual>
-      <collision>
-        <origin rpy="0 0 0" xyz="0.01905 0 0"/>
-         <geometry>
-          <box size="0.0381 .0075 .002"/>
-        </geometry>
-      </collision>
-      <inertial>
-        <origin rpy="0 0 0" xyz="0.01905 -0.00107 0"/>
-        <mass value="0.00538"/>
-        <inertia ixx= "0.00000006639"
-                 ixy="-0.00000010996"
-                 ixz= "0.00000000094"
-                 iyy= "0.00000305318"
-                 iyz= "0"
-                 izz= "0.00000304657"/>
-      </inertial>
-    </link>
-    <gazebo reference="${prefix}link_median_bar">
-      <mu1>1.1</mu1>
-      <mu2>1.1</mu2>
-    </gazebo>
     <!-- Link paramedian hinge -->
-    <link name="${prefix}link_paramedian_hinge">
-      <visual>
-        <origin rpy="0 0 0" xyz="0 0 0"/>
-        <geometry>
-          <box size=".02 .02 .002"/>
-        </geometry>
-      </visual>
-      <collision>
-        <origin rpy="0 0 0" xyz="0 0 0"/>
-         <geometry>
-          <box size=".02 .02 .002"/>
-        </geometry>
-      </collision>
-      <inertial>
-        <origin rpy="0 0 0" xyz="-0.01025 0.00046 0"/>
-        <mass value="0.00276"/>
-        <inertia ixx= "0.00000004213"
-                 ixy="-0.00000001491"
-                 ixz= "0"
-                 iyy= "0.00000050258"
-                 iyz= "0"
-                 izz= "0.00000054007"/>
-      </inertial>
-    </link>
-    <gazebo reference="${prefix}link_paramedian_hinge">
-      <mu1>1.1</mu1>
-      <mu2>1.1</mu2>
-    </gazebo>
     <!-- Link median bar underactuated -->
-    <link name="${prefix}link_median_bar_underactuated">
-      <visual>
-        <origin rpy="0 0 0" xyz="0.01905 0 0"/>
-        <geometry>
-          <box size="0.0381 .0075 .002"/>
-        </geometry>
-      </visual>
-      <collision>
-        <origin rpy="0 0 0" xyz="0.01905 0 0"/>
-         <geometry>
-          <box size="0.0381 .0075 .002"/>
-        </geometry>
-      </collision>
-      <inertial>
-        <origin rpy="0 0 0" xyz="0.01905 -0.00107 0"/>
-        <mass value="0.00538"/>
-        <inertia ixx= "0.00000006639"
-                 ixy="-0.00000010996"
-                 ixz="-0.00000000094"
-                 iyy= "0.00000305318"
-                 iyz= "0"
-                 izz= "0.00000304657"/>
-      </inertial>
-    </link>
-    <gazebo reference="${prefix}link_median_bar_underactuated">
-      <mu1>1.1</mu1>
-      <mu2>1.1</mu2>
-    </gazebo>
     <!-- Link paradistal hinge -->
-    <link name="${prefix}link_paradistal_hinge">
-      <visual>
-        <origin rpy="0 0 0" xyz="0 0 0"/>
-        <geometry>
-          <box size=".02 .02 .002"/>
-        </geometry>
-      </visual>
-      <collision>
-        <origin rpy="0 0 0" xyz="0 0 0"/>
-         <geometry>
-          <box size=".02 0.02 .002"/>
-        </geometry>
-      </collision>
-      <inertial>
-        <origin rpy="0 0 0" xyz="0.00548 0 0"/>
-        <mass value="0.00158"/>
-        <inertia ixx= "0.00000001907"
-                 ixy= "0"
-                 ixz= "0"
-                 iyy= "0.00000010970"
-                 iyz= "0"
-                 izz= "0.00000012610"/>
-      </inertial>
-    </link>
-    <gazebo reference="${prefix}link_paradistal_hinge">
-      <mu1>1.1</mu1>
-      <mu2>1.1</mu2>
-    </gazebo>
     <!-- End of link list -->
     <!-- Joint list -->
     <!-- Joint proximal actuating hinge -->
-    <joint name="${prefix}joint_proximal_actuating_hinge" type="revolute">
-      <parent link="${prefix}link_0"/>
-      <child link="${prefix}link_proximal_actuating_hinge"/>
-      <axis xyz="0 0 1"/>
-      <origin rpy="0 0 -2.0906" xyz="0 0 0.01"/>
-      <limit effort="100" lower="-3.1416" upper="3.1416" velocity="100"/>
-    </joint>
-    <gazebo reference="${prefix}joint_proximal_actuating_hinge">
-      <implicitSpringDamper>1</implicitSpringDamper>
-    </gazebo>
     <!-- Joint paraproximal actuating hinge -->
-    <joint name="${prefix}joint_paraproximal_actuating_hinge" type="revolute">
-      <parent link="${prefix}link_0"/>
-      <child link="${prefix}link_paraproximal_actuating_hinge"/>
-      <axis xyz="0 0 1"/>
-      <origin rpy="0 0 -2.0906" xyz="0 0 -0.01"/>
-      <limit effort="100" lower="-3.1416" upper="3.1416" velocity="100"/>
-    </joint>
-    <gazebo reference="${prefix}joint_paraproximal_actuating_hinge">
-      <implicitSpringDamper>1</implicitSpringDamper>
-    </gazebo>
     <!-- Joint proximal actuating bar -->
-    <joint name="${prefix}joint_proximal_actuating_bar" type="revolute">
-      <parent link="${prefix}link_proximal_actuating_hinge"/>
-      <child link="${prefix}link_proximal_actuating_bar"/>
-      <axis xyz="0 0 1"/>
-      <origin rpy="0 0 1.8616" xyz="0.02858 0 0"/>
-      <limit effort="100" lower="-3.1416" upper="3.1416" velocity="100"/>
-    </joint>
-    <gazebo reference="${prefix}joint_proximal_actuating_bar">
-      <implicitSpringDamper>1</implicitSpringDamper>
-    </gazebo>
     <!-- Joint paraproximal bar -->
-    <joint name="${prefix}joint_paraproximal_bar" type="revolute">
-      <parent link="${prefix}link_paraproximal_actuating_hinge"/>
-      <child link="${prefix}link_paraproximal_bar"/>
-      <axis xyz="0 0 1"/>
-      <origin rpy="0 0 1.57" xyz="0.02286 0 0"/>
-      <limit effort="100" lower="-3.1416" upper="3.1416" velocity="100"/>
-    </joint>
-    <gazebo reference="${prefix}joint_paraproximal_bar">
-      <implicitSpringDamper>1</implicitSpringDamper>
-    </gazebo>
     <!-- Joint median actuating hinge -->
-    <joint name="${prefix}joint_median_actuating_hinge" type="revolute">
-      <parent link="${prefix}link_1"/>
-      <child link="${prefix}link_median_actuating_hinge"/>
-      <axis xyz="0 0 1"/>
-      <origin rpy="0 0 ${-0.37}" xyz="0 0.05715 0.01"/>
-      <limit effort="100" lower="-3.1416" upper="3.1416" velocity="100"/>
-    </joint>
-    <gazebo reference="${prefix}joint_median_actuating_hinge">
-      <implicitSpringDamper>1</implicitSpringDamper>
-    </gazebo>
     <!-- Joint paramedian hinge -->
-    <joint name="${prefix}joint_paramedian_hinge" type="revolute">
-      <parent link="${prefix}link_1"/>
-      <child link="${prefix}link_paramedian_hinge"/>
-      <axis xyz="0 0 1"/>
-      <!-- -0.37 is hand picked, 0.9719 is hand calculated from atan(0.02381/0.01625) -->
-      <origin rpy="0 0 0" xyz="0 0.05715 -0.01"/>
-      <limit effort="100" lower="-3.1416" upper="3.1416" velocity="100"/>
-    </joint>
-    <gazebo reference="${prefix}joint_paramedian_hinge">
-      <implicitSpringDamper>1</implicitSpringDamper>
-    </gazebo>
     <!-- Joint median actuating hinge median bar -->
-    <joint name="${prefix}joint_median_actuating_hinge_median_bar" type="revolute">
-      <parent link="${prefix}link_median_actuating_hinge"/>
-      <child link="${prefix}link_median_bar"/>
-      <axis xyz="0 0 1"/>
-      <!-- hand calc 90 deg + atan(0.01516/0.01625) -->
-      <origin rpy="0 0 ${3.1416/2 + 0.7507}" xyz="0.01625 0.01516 0"/>
-      <limit effort="100" lower="-3.1416" upper="3.1416" velocity="100"/>
-    </joint>
-    <gazebo reference="${prefix}joint_median_actuating_hinge_median_bar">
-      <implicitSpringDamper>1</implicitSpringDamper>
-    </gazebo>
     <!-- Joint paradistal hinge -->
-    <joint name="${prefix}joint_paradistal_hinge" type="revolute">
-      <parent link="${prefix}link_2"/>
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
Commit message: added collision back

File: robotiq/robotiq_s_model_visualization/cfg/robotiq_hand_macro.urdf.xacro (robot description, xacro)
@@ -20,4 +20,13 @@
         </material>
       </visual>
+      <collision>
+        <origin rpy="0 0 0" xyz="0 0 0"/>
+        <geometry>
+          <mesh filename="package://robotiq_s_model_visualization/meshes/s-model_articulated/collision/link_0.STL" />
+        </geometry>
+        <material name="yellow">
+          <color rgba="0 1 1 1"/>
+        </material>
+      </collision>
       <inertial>
         <mass value="0.1"/>
@@ -39,4 +48,13 @@
         <material name="green"/>
       </visual>
+      <collision>
+        <origin rpy="0 0 ${3.1416/2}" xyz="0 0.05717 0"/>
+        <geometry>
+          <mesh filename="package://robotiq_s_model_visualization/meshes/s-model_articulated/collision/link_1.STL"/>
+        </geometry>
+        <material name="yellow">
+          <color rgba="0 1 1 1"/>
+        </material>
+      </collision>
       <inertial>
         <origin rpy="0 0 ${3.1416/2}" xyz="0.00053 0.03218 0"/>
@@ -63,4 +81,11 @@
         <material name="green"/>
       </visual>
+      <collision>
+        <origin rpy="0 0 ${3.1416/2}" xyz="0 0.03810 0.0075"/>
+          <geometry>
+            <mesh filename="package://robotiq_s_model_visualization/meshes/s-model_articulated/collision/link_2.STL"/>
+          </geometry>
+        <material name="yellow"/>
+      </collision>
       <inertial>
         <origin rpy="0 0 ${3.1416/2}" xyz="0.00048 0.02167 0.00018"/>
@@ -77,4 +102,5 @@
       <mu1>1.1</mu1>
       <mu2>1.1</mu2>
+      <self_collide>0</self_collide>
     </gazebo>
     <!-- Link 3 -->
@@ -87,4 +113,11 @@
         <material name="green"/>
       </visual>
+      <collision>
+        <origin xyz="0 0 0" rpy="0 0 0"/>
+        <geometry>
+          <mesh filename="package://robotiq_s_model_visualization/meshes/s-model_articulated/collision/link_3.STL"/>
+        </geometry>
+        <material name="yellow"/>
+      </collision>
       <inertial>
         <origin rpy="0 0 0" xyz="0.01626 0.00049 0.0002"/>
@@ -101,4 +134,5 @@
       <mu1>1.1</mu1>
       <mu2>1.1</mu2>
+      <self_collide>1</self_collide>
     </gazebo>
     <!-- Link proximal actuating hinge -->
@@ -154,5 +188,5 @@
       <dynamics damping="1" friction="0" />
       <axis xyz="0 0 1"/>
-      <origin rpy="0 0 ${3.1416/2 + 0.5198}" xyz="0 0.039 0"/>
+      <origin rpy="0 0 ${3.1416/2 + 0.5198 -0.3}" xyz="0 0.039 0"/>
       <!-- Limits: [-38deg.,60deg.] -->
       <limit lower="-0.6632" upper="1.0471" effort="60" velocity="-1"/>
